Commit message: minor(calib): bagfile and dataset change

File: carbot_calibration/urdf/optimized.urdf.xacro (robot description, xacro)
@@ -1,4 +1,4 @@
-<?xml version="1.0"?>
-<robot name="/home/diogo/catkin_ws/src/robots/carbot/carbot_description/urdf/carbot.urdf" xmlns:xacro="http://ros.org/wiki/xacro">
+<?xml version="1.0" ?>
+<robot name="/home/diogo/catkin_ws/src/robots/carbot/carbot_description/urdf/carbot.urdf" version="1.0">
   <link name="base_link">
     <visual>
@@ -14,9 +14,9 @@
   </link>
   <joint name="wheel4" type="continuous">
+    <origin xyz="-0.05 -0.06 0.0" rpy="1.5708 0.0 0.0"/>
+    <axis xyz="0.0 -4e-06 -1.0"/>
     <parent link="base_link"/>
     <child link="wheel4"/>
-    <axis xyz="0 -0.000004 -1"/>
-    <limit effort="10" velocity="10"/>
-    <origin xyz="-0.05 -0.06 0" rpy="1.5708 0 0"/>
+    <limit effort="10.0" lower="0" upper="0" velocity="10.0"/>
   </joint>
   <link name="wheel4">
@@ -33,9 +33,9 @@
   </link>
   <joint name="wheel3" type="continuous">
+    <origin xyz="-0.05 0.06 0.0" rpy="1.5708 0.0 0.0"/>
+    <axis xyz="0.0 -4e-06 -1.0"/>
     <parent link="base_link"/>
     <child link="wheel3"/>
-    <axis xyz="0 -0.000004 -1"/>
-    <limit effort="10" velocity="10"/>
-    <origin xyz="-0.05 0.06 0" rpy="1.5708 0 0"/>
+    <limit effort="10.0" lower="0" upper="0" velocity="10.0"/>
   </joint>
   <link name="wheel3">
@@ -52,9 +52,9 @@
   </link>
   <joint name="wheel2" type="continuous">
+    <origin xyz="0.05 -0.06 0.0" rpy="1.5708 0.0 0.0"/>
+    <axis xyz="0.0 -4e-06 -1.0"/>
     <parent link="base_link"/>
     <child link="wheel2"/>
-    <axis xyz="0 -0.000004 -1"/>
-    <limit effort="10" velocity="10"/>
-    <origin xyz="0.05 -0.06 0" rpy="1.5708 0 0"/>
+    <limit effort="10.0" lower="0" upper="0" velocity="10.0"/>
   </joint>
   <link name="wheel2">
@@ -71,9 +71,9 @@
   </link>
   <joint name="wheel1" type="continuous">
+    <origin xyz="0.05 0.06 0.0" rpy="1.5708 0.0 0.0"/>
+    <axis xyz="0.0 -4e-06 -1.0"/>
     <parent link="base_link"/>
     <child link="wheel1"/>
-    <axis xyz="0 -0.000004 -1"/>
-    <limit effort="10" velocity="10"/>
-    <origin xyz="0.05 0.06 0" rpy="1.5708 0 0"/>
+    <limit effort="10.0" lower="0" upper="0" velocity="10.0"/>
   </joint>
   <link name="wheel1">
@@ -89,31 +89,27 @@
     </collision>
   </link>
-  <link name="ds_right">
-  </link>
+  <link name="ds_right"/>
   <joint name="base_link_ds_right_joint" type="fixed">
+    <origin xyz="0.105087 -0.032507 0.0" rpy="0.0 0.0 -0.3"/>
     <parent link="base_link"/>
     <child link="ds_right"/>
-    <origin xyz="0.105087 -0.032507 0" rpy="0 0 -0.3"/>
   </joint>
-  <link name="ds_left">
-  </link>
+  <link name="ds_left"/>
   <joint name="base_link_ds_left_joint" type="fixed">
+    <origin xyz="0.105087 0.032507 0.0" rpy="0.0 0.0 0.3"/>
     <parent link="base_link"/>
     <child link="ds_left"/>
-    <origin xyz="0.105087 0.032507 0" rpy="0 0 0.3"/>
   </joint>
-  <link name="accelerometer">
-  </link>
+  <link name="accelerometer"/>
   <joint name="base_link_accelerometer_joint" type="fixed">
+    <origin xyz="0.0062609983603613365 0.0062412830525937655 0.034674001004381415" rpy="0.00999999999999596 -0.009999999999995996 -0.00999999999999596"/>
     <parent link="base_link"/>
     <child link="accelerometer"/>
-    <origin xyz="0 0 0.03" rpy="0 0 0"/>
   </joint>
-  <link name="gyroscope">
-  </link>
+  <link name="gyroscope"/>
   <joint name="base_link_gyroscope_joint" type="fixed">
+    <origin xyz="0.0 0.0 0.03" rpy="0.0 0.0 0.0"/>
     <parent link="base_link"/>
     <child link="gyroscope"/>
-    <origin xyz="0 0 0.03" rpy="0 0 0"/>
   </joint>
 </robot>

File: carbot_description/urdf/carbot.urdf (robot description, URDF)
Before this commit: robot /home/diogo/catkin_ws/src/robots/carbot/carbot_description/urdf/carbot.urdf, 9 links, 8 joints
Links:
- removed link solid
- removed link solid(1)
- removed link solid(1)_0
- added link wheel1; collision cylinder length=0.02 radius=0.04; visual cylinder length=0.02 radius=0.04
- added link wheel3; collision cylinder length=0.02 radius=0.04; visual cylinder length=0.02 radius=0.04
- added link wheel4; collision cylinder length=0.02 radius=0.04; visual cylinder length=0.02 radius=0.04
Joints:
- joint wheel1: child solid -> wheel1
- joint wheel3: child solid(1)_0 -> wheel3
- joint wheel4: child solid(1) -> wheel4

Commit message: fix: fixed a synchronization error which led to bad derivation

File: carbot_calibration/urdf/optimized.urdf.xacro (robot description, xacro)
@@ -1,18 +1,18 @@
 <?xml version="1.0" ?>
-<robot name="/home/diogo/catkin_ws/src/robots/carbot/carbot_description/urdf/carbot.urdf" version="1.0">
+<robot name="/home/diogo/catkin_ws/src/robots/carbot/carbot_description/urdf/carbot2.urdf" version="1.0">
   <link name="base_link">
     <visual>
       <geometry>
-        <box size="0.2 0.1 0.05"/>
+        <box size="0.2 0.1 0.02"/>
       </geometry>
     </visual>
     <collision>
       <geometry>
-        <box size="0.2 0.1 0.05"/>
+        <box size="0.2 0.1 0.02"/>
       </geometry>
     </collision>
   </link>
   <joint name="wheel4" type="continuous">
-    <origin xyz="-0.05 -0.06 0.0" rpy="1.5708 0.0 0.0"/>
+    <origin xyz="-0.05 -0.06 0.0" rpy="1.5708 -1e-06 0.0"/>
     <axis xyz="0.0 -4e-06 -1.0"/>
     <parent link="base_link"/>
@@ -22,4 +22,5 @@
   <link name="wheel4">
     <visual>
+      <origin xyz="-3e-06 2e-06 0.0" rpy="0.0 0.0 0.0"/>
       <geometry>
         <cylinder radius="0.04" length="0.02"/>
@@ -27,4 +28,5 @@
     </visual>
     <collision>
+      <origin xyz="-3e-06 2e-06 0.0" rpy="0.0 0.0 0.0"/>
       <geometry>
         <cylinder radius="0.04" length="0.02"/>
@@ -33,5 +35,5 @@
   </link>
   <joint name="wheel3" type="continuous">
-    <origin xyz="-0.05 0.06 0.0" rpy="1.5708 0.0 0.0"/>
+    <origin xyz="-0.050003 0.060002 0.0" rpy="1.5708 0.0 0.0"/>
     <axis xyz="0.0 -4e-06 -1.0"/>
     <parent link="base_link"/>
@@ -41,4 +43,5 @@
   <link name="wheel3">
     <visual>
+      <origin xyz="0.0 5e-06 0.0" rpy="0.0 0.0 0.0"/>
       <geometry>
         <cylinder radius="0.04" length="0.02"/>
@@ -46,4 +49,5 @@
     </visual>
     <collision>
+      <origin xyz="0.0 5e-06 0.0" rpy="0.0 0.0 0.0"/>
       <geometry>
         <cylinder radius="0.04" length="0.02"/>
@@ -52,5 +56,5 @@
   </link>
   <joint name="wheel2" type="continuous">
-    <origin xyz="0.05 -0.06 0.0" rpy="1.5708 0.0 0.0"/>
+    <origin xyz="0.05 -0.059995 0.0" rpy="1.5708 -1e-06 0.0"/>
     <axis xyz="0.0 -4e-06 -1.0"/>
     <parent link="base_link"/>
@@ -60,4 +64,5 @@
   <link name="wheel2">
     <visual>
+      <origin xyz="-3e-06 2e-06 0.0" rpy="0.0 0.0 0.0"/>
       <geometry>
         <cylinder radius="0.04" length="0.02"/>
@@ -65,4 +70,5 @@
     </visual>
     <collision>
+      <origin xyz="-3e-06 2e-06 0.0" rpy="0.0 0.0 0.0"/>
       <geometry>
         <cylinder radius="0.04" length="0.02"/>
@@ -71,5 +77,5 @@
   </link>
   <joint name="wheel1" type="continuous">
-    <origin xyz="0.05 0.06 0.0" rpy="1.5708 0.0 0.0"/>
+    <origin xyz="0.049997 0.060002 0.0" rpy="1.5708 0.0 0.0"/>
     <axis xyz="0.0 -4e-06 -1.0"/>
     <parent link="base_link"/>
@@ -79,4 +85,5 @@
   <link name="wheel1">
     <visual>
+      <origin xyz="0.0 5e-06 0.0" rpy="0.0 0.0 0.0"/>
       <geometry>
         <cylinder radius="0.04" length="0.02"/>
@@ -84,4 +91,5 @@
     </visual>
     <collision>
+      <origin xyz="0.0 5e-06 0.0" rpy="0.0 0.0 0.0"/>
       <geometry>
         <cylinder radius="0.04" length="0.02"/>
@@ -91,5 +99,5 @@
   <link name="ds_right"/>
   <joint name="base_link_ds_right_joint" type="fixed">
-    <origin xyz="0.105087 -0.032507 0.0" rpy="0.0 0.0 -0.3"/>
+    <origin xyz="0.105087 -0.032502 0.0" rpy="0.0 0.0 -0.3"/>
     <parent link="base_link"/>
     <child link="ds_right"/>
@@ -101,15 +109,32 @@
     <child link="ds_left"/>
   </joint>
+  <link name="gyro"/>
+  <joint name="base_link_gyro_joint" type="fixed">
+    <origin xyz="0.0 0.0 0.015" rpy="0.0 0.0 0.0"/>
+    <parent link="base_link"/>
+    <child link="gyro"/>
+  </joint>
   <link name="accelerometer"/>
   <joint name="base_link_accelerometer_joint" type="fixed">
-    <origin xyz="0.0062609983603613365 0.0062412830525937655 0.034674001004381415" rpy="0.00999999999999596 -0.009999999999995996 -0.00999999999999596"/>
+    <origin xyz="0.0008244156733916555 0.00049225321909848 0.014995792462240684" rpy="-3.668874226961156e-05 -7.769112709439543e-05 -0.0007952407141155575"/>
     <parent link="base_link"/>
     <child link="accelerometer"/>
   </joint>
-  <link name="gyroscope"/>
-  <joint name="base_link_gyroscope_joint" type="fixed">
-    <origin xyz="0.0 0.0 0.03" rpy="0.0 0.0 0.0"/>
+  <link name="solid">
+    <visual>
+      <geometry>
+        <box size="0.2 0.1 0.02"/>
+      </geometry>
+    </visual>
+    <collision>
+      <geometry>
+        <box size="0.2 0.1 0.02"/>
+      </geometry>
+    </collision>
+  </link>
+  <joint name="base_link_solid_joint" type="fixed">
+    <origin xyz="0.0 0.0 0.0" rpy="0.0 0.0 0.0"/>
     <parent link="base_link"/>
-    <child link="gyroscope"/>
+    <child link="solid"/>
   </joint>
 </robot>
